File: Commiepad V2 PCB/Commiepad V2.kicad_pcb (KiCad board)
At the start: 2 copper layers, 85.6 x 64.4 mm, 29 parts, among them J1 SSD1306 OLED, SW1 RotaryEncoder_Switch_MP, SW2 SW_Push_45deg, SW3 SW_Push_45deg, SW4 SW_Push_45deg, SW5 SW_Push_45deg, SW6 SW_Push_45deg, SW7 SW_Push_45deg, SW8 SW_Push_45deg, SW9 SW_Push_45deg, U1 XIAO-RP2040-DIP

Commit message: Added PCB, CAD files and edited the README
Changed lines of the file:
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@@
 		)
 		(embedded_fonts no)
-		(model "W:/Commiepad V2 Footprints/Seeed Studio XIAO RP2040 v26.step"
+		(model "C:/Users/Adiptoo/Downloads/seeed-studio-xiao-rp2040-3d-model/Seeed Studio XIAO RP2040 v26.step"
 			(offset
 				(xyz 0 0 0)
@@
 		(polygon
 			(pts
-				(xy 112.685418 37.832919) (xy 212.23 36.97) (xy 213.46 109.5) (xy 106.554294 108.630417)
+				(xy 123.83 40.75) (xy 209.79 40.98) (xy 209.592978 106.66039) (xy 122.902143 106.400343)
 			)
 		)
@@
 		(polygon
 			(pts
-				(xy 118.79 37.78) (xy 212.23 36.97) (xy 213.46 109.5) (xy 112.65 108.68)
+				(xy 123.47 40.51) (xy 209.91 40.75) (xy 209.284555 106.772933) (xy 123.47 105.96)
 			)
 		)
