File: Commiepad V2 PCB/Commiepad V2.kicad_sch (KiCad schematic)
At the start: 28 parts, among them J1 SSD1306 OLED, SW1 RotaryEncoder_Switch_MP, SW2 SW_Push_45deg, SW3 SW_Push_45deg, SW4 SW_Push_45deg, SW5 SW_Push_45deg, SW6 SW_Push_45deg, SW7 SW_Push_45deg, SW8 SW_Push_45deg, SW9 SW_Push_45deg, U1 XIAO-RP2040-DIP

Commit message: Added PCB, CAD files and edited the README
Other:
- company: (none) -> Hasnat4763.me
- title: (none) -> Commiepad
Changed lines of the file:
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@@
 	(generator_version "10.0")
 	(paper "A3")
+	(title_block
+		(title "Commiepad")
+		(date "2026-05-17")
+		(rev " V2")
+		(company "Hasnat4763.me")
+	)
 	(rectangle
 		(start 20.32 144.272)
